File: UPX_Port_Adapter.brd (EAGLE design)
At the start: 120.3 x 89 mm, 35 parts, among them J1 SM02BGHSTBLFSN, J10 SM07B-GHS-TB(LF)(SN), J11 SM07B-GHS-TB(LF)(SN), J12 SM04B-GHS-TB(LF)(SN)-, J13 SM04B-GHS-TB(LF)(SN)-, J2 SM02BGHSTBLFSN, J3 SM02BGHSTBLFSN, J4 SM02BGHSTBLFSN, J5 SM02BGHSTBLFSN, J6 SM02BGHSTBLFSN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

Commit message: Traces Reviewed
Routing:
- net 3V3: track 182.1 -> 204.3 mm, vias 0 -> 1
- net SCK1: track 61.0 -> 62.8 mm
- net GND: vias 23 -> 39
Changed lines of the file:
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@@
 </polygon>
 <via x="76" y="72" extent="1-16" drill="0.35"/>
-<via x="72" y="76" extent="1-16" drill="0.35"/>
+<via x="71.75" y="80" extent="1-16" drill="0.35"/>
 <via x="87" y="77" extent="1-16" drill="0.35"/>
 <via x="96" y="77" extent="1-16" drill="0.35"/>
@@
 <via x="48.5" y="1.5" extent="1-16" drill="0.35"/>
 <via x="51" y="1.5" extent="1-16" drill="0.35"/>
+<via x="95.25" y="70" extent="1-16" drill="0.35"/>
+<via x="95.5" y="61" extent="1-16" drill="0.35"/>
+<via x="95.5" y="52.75" extent="1-16" drill="0.35"/>
+<via x="95.5" y="45" extent="1-16" drill="0.35"/>
+<via x="95.5" y="37.25" extent="1-16" drill="0.35"/>
+<via x="95.5" y="29" extent="1-16" drill="0.35"/>
+<via x="95.5" y="20.75" extent="1-16" drill="0.35"/>
+<via x="95.75" y="13" extent="1-16" drill="0.35"/>
+<via x="95.75" y="5.5" extent="1-16" drill="0.35"/>
+<via x="34.25" y="70" extent="1-16" drill="0.35"/>
+<via x="75" y="69" extent="1-16" drill="0.35"/>
+<via x="53.75" y="70" extent="1-16" drill="0.35"/>
+<via x="19.75" y="68" extent="1-16" drill="0.35"/>
+<via x="18.25" y="70.75" extent="1-16" drill="0.35"/>
+<via x="13" y="68" extent="1-16" drill="0.35"/>
+<via x="67.75" y="76.75" extent="1-16" drill="0.35"/>
 </signal>
 <signal name="SDA_3V3">
@@
 <wire x1="67.4" y1="70.05" x2="65.9" y2="68.55" width="0.3048" layer="1"/>
 <wire x1="65.9" y1="68.55" x2="59.4" y2="68.55" width="0.3048" layer="1"/>
-<wire x1="11.19" y1="33.96" x2="13.46" y2="33.96" width="0.3048" layer="1"/>
+<wire x1="11.19" y1="33.96" x2="11.21" y2="33.96" width="0.3048" layer="1"/>
 <wire x1="22.55" y1="68.55" x2="59.4" y2="68.55" width="0.3048" layer="1"/>
-<wire x1="13.46" y1="33.96" x2="19" y2="39.5" width="0.3048" layer="1"/>
-<wire x1="19" y1="39.5" x2="19" y2="65" width="0.3048" layer="1"/>
+<wire x1="11.21" y1="33.96" x2="19" y2="41.75" width="0.3048" layer="1"/>
+<wire x1="19" y1="41.75" x2="19" y2="65" width="0.3048" layer="1"/>
 <wire x1="19" y1="65" x2="22.55" y2="68.55" width="0.3048" layer="1"/>
 <contactref element="J12" pad="3"/>
@@
 <wire x1="6.7" y1="5.8" x2="6.75" y2="5.8" width="0.2032" layer="1"/>
 <wire x1="6.5" y1="5.6" x2="6.75" y2="5.35" width="0.2032" layer="1"/>
-<wire x1="11.19" y1="13.64" x2="11.19" y2="33.96" width="0" layer="19" extent="1-1"/>
+<wire x1="11.19" y1="13.64" x2="13.14" y2="13.64" width="0.508" layer="16"/>
+<wire x1="13.14" y1="13.64" x2="13.75" y2="14.25" width="0.508" layer="16"/>
+<via x="13.75" y="14.25" extent="1-16" drill="0.35"/>
+<wire x1="13.75" y1="14.25" x2="13.75" y2="31.4" width="0.508" layer="1"/>
+<wire x1="13.75" y1="31.4" x2="11.19" y2="33.96" width="0.508" layer="1"/>
 </signal>
 <signal name="5V">
@@
 <contactref element="JP2" pad="18"/>
 <wire x1="9.91" y1="40.3" x2="11.19" y2="41.58" width="0.2032" layer="1"/>
-<wire x1="6.32" y1="40.3" x2="9.91" y2="40.3" width="0.2032" layer="1"/>
+<wire x1="9.91" y1="40.3" x2="6.32" y2="40.3" width="0.2032" layer="1"/>
 <contactref element="J11" pad="3"/>
 <wire x1="33.5" y1="4.6" x2="33.5" y2="8.75" width="0.1524" layer="1"/>
@@
 <wire x1="22.5" y1="40.25" x2="12.52" y2="40.25" width="0.1524" layer="16"/>
 <wire x1="12.52" y1="40.25" x2="11.19" y2="41.58" width="0.1524" layer="16"/>
-<wire x1="6.32" y1="40.3" x2="5.04" y2="41.58" width="0" layer="19" extent="1-1"/>
+<wire x1="6.32" y1="40.3" x2="5.04" y2="41.58" width="0.2032" layer="1"/>
 </signal>
 <signal name="MOSI2">
@@
 <wire x1="3.76915625" y1="40.306" x2="5.46084375" y2="40.306" width="0.2032" layer="1"/>
 <wire x1="6.72684375" y1="39.04" x2="8.65" y2="39.04" width="0.2032" layer="1"/>
-<wire x1="2.50315625" y1="39.04" x2="3.76915625" y2="40.306" width="0.2032" layer="1"/>
+<wire x1="2.75315625" y1="39.29" x2="3.76915625" y2="40.306" width="0.2032" layer="1"/>
 <wire x1="5.46084375" y1="40.306" x2="6.72684375" y2="39.04" width="0.2032" layer="1"/>
 <contactref element="J10" pad="1"/>
@@
 <wire x1="9.9" y1="37.79" x2="8.65" y2="39.04" width="0.1524" layer="16"/>
 <wire x1="9.9" y1="35.85" x2="9.9" y2="37.79" width="0.1524" layer="16"/>
-<wire x1="2.50315625" y1="39.04" x2="2.5" y2="39.04" width="0" layer="19" extent="1-1"/>
+<wire x1="2.5" y1="39.04" x2="2.75" y2="39.29" width="0.2032" layer="1"/>
+<wire x1="2.75" y1="39.29" x2="2.75315625" y2="39.29" width="0.2032" layer="1"/>
 </signal>
 <signal name="SCK2">
@@
 <mfgpreviewcolor name="substratecolor" color="0xFF3C3D30"/>
 </mfgpreviewcolors>
+<errors>
+</errors>
 </board>
 </drawing>

Commit message: Added mfg files and visuals
Parts:
- C1, C2, C3, C4: device rcl:C0603 -> UPX_Port_Adapter:RCL_C0603
- J1, J2, J3, J4, J5, J6, J7, J8, J9: value SM02BGHSTBLFSN -> SM02B-GHS-TB_SM02BGHSTBLFSN; device SM02B-GHS-TB:CONN_SM02BGHSTB_JST -> UPX_Port_Adapter:SM02B-GHS-TB_CONN_SM02BGHSTB_JST
- J10, J11: value SM07B-GHS-TB(LF)(SN) -> SM07B-GHS-TB_LF__SN__SM07B-GHS-TB(LF)(SN); device SM07B-GHS-TB_LF__SN_:JST_SM07B-GHS-TB(LF)(SN) -> UPX_Port_Adapter:SM07B-GHS-TB_LF__SN__JST_SM07B-GHS-TB(LF)(SN)
- J12, J13: value SM04B-GHS-TB(LF)(SN)- -> SM04B-GHS-TB_LF__SN_-_SM04B-GHS-TB(LF)(SN)-; device SM04B-GHS-TB_LF__SN_-:JST_SM04B-GHS-TB(LF)(SN)- -> UPX_Port_Adapter:SM04B-GHS-TB_LF__SN_-_JST_SM04B-GHS-TB(LF)(SN)-
- JP1: device pinhead:2X20 -> UPX_Port_Adapter:PINHEAD_2X20
- JP2: device pinhead2:2X20/90 -> UPX_Port_Adapter:PINHEAD2_2X20/90
- R1, R2, R3, R4, R5, R6: device rcl:R0603 -> UPX_Port_Adapter:RCL_R0603
- U$1, U$2, U$3, U$4, U$5, U$6, U$7, U$8: value PCAN_CONN -> SM05B-SURS-TF_LF__SN__PCAN_CONN; device SM05B-SURS-TF_LF__SN_:SM05BSURSTFLFSN -> UPX_Port_Adapter:SM05B-SURS-TF_LF__SN__SM05BSURSTFLFSN
- U$9: value 20X20 -> PINHEAD-CUSTOM_20X20; device pinhead-CUSTOM:20X20 -> UPX_Port_Adapter:PINHEAD-CUSTOM_20X20
- U1: value NLSX3012DR2G -> NLSX3012DR2G_NLSX3012DR2G; device NLSX3012DR2G:SOIC-8_NB_ONS -> UPX_Port_Adapter:NLSX3012DR2G_SOIC-8_NB_ONS
