File: UPX_Port_Adapter.sch (EAGLE design)
At the start: 35 parts, among them J1 SM02BGHSTBLFSN, J10 SM07B-GHS-TB(LF)(SN), J11 SM07B-GHS-TB(LF)(SN), J12 SM04B-GHS-TB(LF)(SN)-, J13 SM04B-GHS-TB(LF)(SN)-, J2 SM02BGHSTBLFSN, J3 SM02BGHSTBLFSN, J4 SM02BGHSTBLFSN, J5 SM02BGHSTBLFSN, J6 SM02BGHSTBLFSN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

Commit message: Added mfg files and visuals
Parts:
- C1, C2, C3, C4: device rcl:C-EUC0603 -> UPX_Port_Adapter:RCL_C-EUC0603
- J1, J2, J3, J4, J5, J6, J7, J8, J9: value SM02BGHSTBLFSN -> SM02B-GHS-TB_SM02BGHSTBLFSN; device SM02B-GHS-TB:SM02BGHSTBLFSN -> UPX_Port_Adapter:SM02B-GHS-TB_SM02BGHSTBLFSN
- J10, J11: value SM07B-GHS-TB(LF)(SN) -> SM07B-GHS-TB_LF__SN__SM07B-GHS-TB(LF)(SN); device SM07B-GHS-TB_LF__SN_:SM07B-GHS-TB(LF)(SN) -> UPX_Port_Adapter:SM07B-GHS-TB_LF__SN__SM07B-GHS-TB(LF)(SN)
- J12, J13: value SM04B-GHS-TB(LF)(SN)- -> SM04B-GHS-TB_LF__SN_-_SM04B-GHS-TB(LF)(SN)-; device SM04B-GHS-TB_LF__SN_-:SM04B-GHS-TB(LF)(SN)- -> UPX_Port_Adapter:SM04B-GHS-TB_LF__SN_-_SM04B-GHS-TB(LF)(SN)-
- JP1: device pinhead:PINHD-2X20 -> UPX_Port_Adapter:PINHEAD_PINHD-2X20
- JP2: device pinhead2:PINHD-2X20/90 -> UPX_Port_Adapter:PINHEAD2_PINHD-2X20/90:1
- R1, R2, R3, R4, R5, R6: device rcl:R-US_R0603 -> UPX_Port_Adapter:RCL_R-US_R0603
- U$1, U$2, U$3, U$4, U$5, U$6, U$7, U$8: value PCAN_CONN -> SM05B-SURS-TF_LF__SN__PCAN_CONN; device SM05B-SURS-TF_LF__SN_:PCAN_CONN -> UPX_Port_Adapter:SM05B-SURS-TF_LF__SN__PCAN_CONN
- U$9: value 20X20 -> PINHEAD-CUSTOM_20X20; device pinhead-CUSTOM:20X20 -> UPX_Port_Adapter:PINHEAD-CUSTOM_20X20
- U1: value NLSX3012DR2G -> NLSX3012DR2G_NLSX3012DR2G; device NLSX3012DR2G:NLSX3012DR2G -> UPX_Port_Adapter:NLSX3012DR2G_NLSX3012DR2G
